File: I2C_Bus_1.kicad_sch (KiCad schematic)
At the start: 8 parts, among them U3 ICM-42688-P, U6 SHT4x

Commit message: major routing update!
Parts:
- R18, R21: value 1k -> 1K
Changed lines of the file:
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@@
 			)
 		)
-		(property "Value" "1k"
+		(property "Value" "1K"
 			(at 211.836 115.57 0)
 			(effects
@@
 			)
 		)
-		(property "Value" "1k"
+		(property "Value" "1K"
 			(at 219.456 115.57 0)
 			(effects
