File: flight-computer-lite.kicad_pcb (KiCad board)
At the start: 2 copper layers, 65 x 65 mm, 94 parts, among them J1 USB_C_Receptacle_USB2.0_16P, J2 Micro_SD_Card_Det2, J3 Conn_01x02_Pin, J4 Conn_01x03_Pin, Q1 NX3008NBK,215, Q2 NX3008NBK,215, SW1 SW_Push, SW2 SW_Push, U1 RP2040, U11 LM66200DRLR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

Commit message: Moved back silkscreen
Parts:
- moved G*** 112.3 mm to (53.4, 51.9)
- moved G*** 112.3 mm to (40.1, 25.7)

Commit message: Design complete (hopefully)
Parts:
- U5: footprint Package_LGA:LGA-12_2x2mm_P0.5mm -> LRI_partlib:LGA-12_2x2mm_P0.5mm
Connections:
- AE1 pad 2: (no net) -> GND
- J4 pad MP: (no net) -> GND
